File: board/stm32h755xih3/stm32h755xih3.kicad_sch (KiCad schematic)
At the start: 75 parts, among them IC1 USBLC6-2SC6, IC2 USBLC6-2SC6, IC3 USBLC6-2SC6, IC4 USBLC6-2SC6, IC5 USBLC6-2SC6, IC6 USBLC6-2SC6, IC7 USBLC6-2SC6, IC8 TPS629203QDRLRQ1, IC9 AP2112K-3.3TRG1, J1 HTSW-101-07-G-T, J10 HTSW-101-07-G-T, J11 HTSW-101-07-G-T, J12 HTSW-101-07-G-T, J13 HTSW-101-07-G-T, J14 HTSW-101-07-G-T, J15 HTSW-101-07-G-T, J16 HTSW-101-07-G-T, J17 HTSW-101-07-G-T, J18 Conn_ARM_SWD_TagConnect_TC203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, J2 HTSW-101-07-G-T, J3 HTSW-101-07-G-T, J4 BM06B-GHS-GB-TBT_LF__SN_, J5 BM06B-GHS-GB-TBT_LF__SN_, J6 BM06B-GHS-GB-TBT_LF__SN_, J7 HTSW-101-07-G-T, J8 HTSW-101-07-G-T, J9 10155435-00011LF, U1 STM32H755ZITx, Y1 LFXTAL085880

Commit message: pcb update
Parts:
- removed C1: MLASG168BB5475KTNA01, CAPC1709X100N, symbol MLASG168BB5475KTNA01:MLASG168BB5475KTNA01
- removed C29: CC0603JRX7R9BB104, CAPC1608X90N, symbol CC0603JRX7R9BB104:CC0603JRX7R9BB104
- removed C4: CL31A226KOCLNNC, CAPC3216X95N, symbol CL31A226KOCLNNC:CL31A226KOCLNNC
- removed D1, D2: MBR0530T1G, SOD3716X135N, symbol MBR0530T1G:MBR0530T1G
- removed IC1, IC2, IC3, IC4, IC5, IC6, IC7: USBLC6-2SC6, SOT95P280X145-6N, symbol USBLC6-2SC6:USBLC6-2SC6
- removed IC8: TPS629203QDRLRQ1, SOTFL50P160X60-8N, symbol TPS629203QDRLRQ1:TPS629203QDRLRQ1
- removed J1: HTSW-101-07-G-T, HDRV3W64P254_3X1_254X756X838P, symbol HTSW-101-07-G-T:HTSW-101-07-G-T
- removed J5, J6: BM06B-GHS-GB-TBT_LF__SN_, BM06BGHSGBTBTLFSN, symbol BM06B-GHS-GB-TBT_LF__SN_:BM06B-GHS-GB-TBT_LF__SN_
- removed J9: 10155435-00011LF, 10155435-00011LF:AMPHENOL_10155435-00011LF, symbol 10155435-00011LF:10155435-00011LF
- removed L1: SRP3212-2R2M, INDC2520X100N, symbol SRP3212-2R2M:SRP3212-2R2M
- removed R1, R3: CRCW01005K10FREL, RESC0402X15N, symbol CRCW01005K10FREL:CRCW01005K10FREL
- removed R2: CRCW040227K4FKED, CRCW0402200KFKED, symbol CRCW040227K4FKED:CRCW040227K4FKED
- added C28, C6: CC0603JRX7R9BB104, CAPC1608X90N, symbol CC0603JRX7R9BB104:CC0603JRX7R9BB104
- added C4: KGM31HR71C105JU, CAPC3216X190N, symbol KGM31HR71C105JU:KGM31HR71C105JU
- added J14, J9: BM06B-GHS-GB-TBT_LF__SN_, BM06BGHSGBTBTLFSN, symbol BM06B-GHS-GB-TBT_LF__SN_:BM06B-GHS-GB-TBT_LF__SN_
- added J17, J4: HTSW-101-07-G-T, HDRV3W64P254_3X1_254X756X838P, symbol HTSW-101-07-G-T:HTSW-101-07-G-T
- added TP1, TP10, TP11, TP12, TP13, TP14, TP15, TP2, TP3, TP4, TP5, TP6, TP7, TP8, TP9: TestPoint, symbol Connector:TestPoint
- renumbered C2 to C1, C11 to C10, C12 to C11, C13 to C12, C9 to C13, C16 to C15, C18 to C16, C15 to C17, C19 to C18, C17 to C19, C3 to C2, C27 to C26, C26 to C27, C28 to C29, C5 to C3, C33 to C32, C32 to C33, C6 to C5, C8 to C7, C10 to C8, C7 to C9, IC9 to IC1, J4 to J1, J12 to J10, J13 to J11, J14 to J12, J15 to J13, J16 to J15, J17 to J16, J7 to J5, J8 to J6, J10 to J7, J11 to J8, L2 to L1, R4 to R1, R5 to R2, R6 to R3, R7 to R4
Connections:
- net 3V3USB is gone; now on net 3V3: C26.1, U1.91 (VDD33_USB)
- net D- is gone; now on net STM32D1/2: U1.101 (PA12)
- net STM32E is gone; now on net STM32E1/2: J16.1, U1.86 (PG6)
- net 3V3: now also C3.1, IC1.5 (VOUT), C28.1, C4.1, C6.1, TP14.1
- net APU1A: now also TP1.1
- net APU1B: now also TP4.1
- net APU1C: now also TP2.1
- net APU1D: now also TP5.1
- net APU2A: now also TP6.1
- net APU2B: now also TP8.1
- net APU2C: now also TP7.1
- net APU2D: now also TP9.1
- net GND: now also C28.2, C4.2, C6.2, J14.6, J14.7 (MP1), J14.8 (MP2), J17.3, J4.3, J9.6, J9.7 (MP1), J9.8 (MP2)
- net RXD1: now also J1.3, U1.134 (PB7); no longer U1.120 (PD6)
- net RXD2: now also U1.120 (PD6), J9.3; no longer U1.122 (PG9)
- net RXD3: now also U1.110 (PC11), J14.3; no longer U1.20 (PF6)
- net TXD1: now also J1.2, U1.133 (PB6); no longer U1.117 (PD5)
- net TXD2: now also U1.117 (PD5), J9.2; no longer U1.127 (PG14)
- net TXD3: now also U1.109 (PC10), J14.2; no longer U1.21 (PF7)
- net STM32E1/2: now reaches U1.87 (PG7)
- net STM32E1/2: now also TP13.1
- net STM32Α1/2: now reaches U1.94 (PC7)
- net STM32Α1/2: now also J12.1, TP10.1
- net STM32B1/2: now reaches U1.97 (PA8)
- net STM32B1/2: now also J15.1, U1.95 (PC8), TP12.1
- net STM32C1/2: now reaches U1.99 (PA10)
- net STM32C1/2: now also U1.98 (PA9), J17.1, TP15.1
- net CTS1: no longer names the net of U1.115 (PD3)
- net CTS2: no longer names the net of U1.126 (PG13)
- net CTS3: no longer names the net of U1.23 (PF9)
- net D+ renamed STM32D1/2
- net STM32D1/2: now also TP11.1
- net RTS1: no longer names the net of U1.116 (PD4)
- net RTS2: no longer names the net of U1.125 (PG12)
- net RTS3: no longer names the net of U1.22 (PF8)
- removed net STM32B: J12.1, U1.95 (PC8)
- removed net STM32C: J15.1, U1.98 (PA9)
- net VBUS: no longer names the net of C1.1, C2.1, IC1.1 (VIN), IC1.3 (EN)
- net VBUS: now also J4.1, TP3.1; no longer U1.90 (VDD50_USB)
- net VCAP: no longer names the net of C19.1, U1.103 (VCAP), U1.140 (VCAP)
- net VCAP: no longer C17.1, U1.68 (VCAP)
- new net: C17.1, U1.68 (VCAP)
- no-connect marks 20 -> 96
Other:
- company: (none) -> SAVILO-AKATE PRODUCTIONS
- title: (none) -> APU-MUX
- moved on the sheet: C1, C10, C11, C12, C13, C14, C15, C16, C17, C18, C19, C2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

Commit message: board updates
Parts:
- removed C13: GRM188R61A106KE69D, CAPC1608X90N, symbol GRM188R61A106KE69D:GRM188R61A106KE69D
- removed C22: MLASG168BB5475KTNA01, CAPC1709X100N, symbol MLASG168BB5475KTNA01:MLASG168BB5475KTNA01
- removed C31, C33: 06035C3R9CAT2A, CAPC1608X90N, symbol 06035C3R9CAT2A:06035C3R9CAT2A
- removed C9: GRM1885C1H221JA01D, CAPC1608X90N, symbol GRM1885C1H221JA01D:GRM1885C1H221JA01D
- removed J1, J14, J9: BM06B-GHS-GB-TBT_LF__SN_, BM06BGHSGBTBTLFSN, symbol BM06B-GHS-GB-TBT_LF__SN_:BM06B-GHS-GB-TBT_LF__SN_
- removed J18: Conn_ARM_SWD_TagConnect_TC2030-NL, Connector:Tag-Connect_TC2030-IDC-NL_2x03_P1.27mm_Vertical, symbol Connector:Conn_ARM_SWD_TagConnect_TC2030-NL
- removed L1: SRP3212-2R2M, INDC2520X100N, symbol SRP3212-2R2M:SRP3212-2R2M
- added C26, C28: GRM1555C1H8R0DA01D, CAPC1005X70N, symbol GRM1555C1H8R0DA01D:GRM1555C1H8R0DA01D
- added J11, J17, J18, J6: 205957-0671, 2059570671, symbol 205957-0671:205957-0671
- renumbered C11 to C10, C12 to C11, C25 to C12, C14 to C13, C15 to C14, C16 to C15, C18 to C16, C27 to C17, C20 to C18, C29 to C19, C21 to C20, C30 to C21, C23 to C22, C24 to C23, C26 to C24, C28 to C25, C32 to C27, C19 to C29, C17 to C30, C5 to C4, C7 to C5, C4 to C6, C8 to C7, C6 to C8, C10 to C9, J2 to J1, J11 to J10, J15 to J14, J16 to J15, J17 to J16, J3 to J2, J4 to J3, J5 to J4, J6 to J5, J10 to J9
Connections:
- net VFBSMPS is gone; now on net GND: U1.17 (VFBSMPS)
- net 3V3: now also J18.1; no longer U1.16 (VDDSMPS)
- net GND: now also U1.16 (VDDSMPS), C26.2, C28.1, J11.1, J11.MP1, J11.MP2, J17.1, J17.MP1, J17.MP2, J18.6, J18.MP1, J18.MP2, J6.1, J6.MP1, J6.MP2
- net NRESET: now also J18.2
- net OSC1: now also C28.2
- net OSC2: now also C26.1
- net RXD1: now also J6.4
- net RXD2: now also J11.4
- net RXD3: now also J17.4
- net SWCLK: now also J18.3
- net SWDIO: now also J18.4
- net SWO: now also J18.5
- net TXD1: now also J6.5
- net TXD2: now also J11.5
- net TXD3: now also J17.5
- net APU1A renamed AP1_1
- net APU1B renamed AP1_2
- net AP1_2: no longer U1.108 (PA15)
- net APU1C renamed AP1_3
- net APU1D renamed AP1_4
- net APU2A renamed AP2_1
- net APU2B renamed AP2_2
- net APU2C renamed AP2_3
- net APU2D renamed AP2_4
- net VLXSMPS: no longer names the net of U1.15 (VLXSMPS)
- new net APU1_2: U1.108 (PA15)
- no-connect marks 96 -> 97
Other:
- note added: "mates with: 2045320601"
- moved on the sheet: C10, C11, C12, C13, C14, C15, C16, C17, C18, C19, C20, C21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

Commit message: board final???
Parts:
- removed C12: CC0603JRX7R9BB104, C35, symbol CC0603JRX7R9BB104:CC0603JRX7R9BB104
- removed C17, C19, C2, C21, C24, C3, C6: KGM31HR71C105JU, CAPC3216X190N, symbol KGM31HR71C105JU:KGM31HR71C105JU
- removed C25: CC0603JRX7R9BB104, CAPC1608X90N, symbol CC0603JRX7R9BB104:CC0603JRX7R9BB104
- removed J11, J17, J18, J6: 205957-0671, 2059570671, symbol 205957-0671:205957-0671
- removed Y1: LFXTAL085880, LFXTAL085880, symbol LFXTAL085880:LFXTAL085880
- added C14: CC0603JRX7R9BB104, CAPC1608X90N, symbol CC0603JRX7R9BB104:CC0603JRX7R9BB104
- added C19, C2, C21, C23, C3, C8: C0603X105J4RACTU, C0603, symbol C0603X105J4RACTU:C0603X105J4RACTU
- added J14, J18, J4, J9: 53047-0610, 530470610, symbol 53047-0610:53047-0610
- added Y1: 830059082, 830059082, symbol 830059082:830059082
- renumbered C11 to C10, C8 to C11, C13 to C12, C14 to C13, C18 to C17, C20 to C18, C22 to C20, C23 to C22, C26 to C24, C27 to C25, C28 to C26, C29 to C27, C30 to C28, C5 to C4, C4 to C5, C7 to C6, C9 to C7, C10 to C9, J9 to J10, J10 to J11, J14 to J15, J15 to J16, J16 to J17, J4 to J5, J5 to J6
Connections:
- net APU1_2 is gone; now on net AP1_2: U1.108 (PA15)
- net 3V3: now also U1.90 (VDD50_USB), C14.1, C19.1, C21.1, C23.1, C3.2, C8.1, J18.1
- net GND: now also C14.2, C19.2, C2.1, C21.2, C23.2, C3.1, C8.2, J14.1, J18.6, J4.1, J9.1, Y1.2 (GND_&_LID_1), Y1.4 (GND_&_LID_2)
- net NRESET: now also J18.2
- net OSC1: now also Y1.1 (CRYSTAL_1)
- net OSC2: now also Y1.3 (CRYSTAL_2)
- net RXD1: now also J4.4
- net RXD2: now also J9.4
- net RXD3: now also J14.4
- net SWCLK: now also J18.3
- net SWDIO: now also J18.4
- net SWO: now also J18.5
- net TXD1: now also J4.5
- net TXD2: now also J9.5
- net TXD3: now also J14.5
- net at C1.1, IC1.1 (VIN), IC1.3 (EN)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: now also C2.2
- no-connect marks 97 -> 96
Other:
- note added: "mates with: 510210600"
- note removed: "mates with: 2045320601"
- moved on the sheet: C11, C26, C5

Commit message: final??
Parts:
- removed C27, C28: 12065C225JAT2A, CAPC3216X229N, symbol 12065C225JAT2A:12065C225JAT2A
- added C27, C28: 0603YC225MAT2A, CAPC1608X90N, symbol 0603YC225MAT2A:0603YC225MAT2A
Connections:
- net GND: now also C27.1, C28.1
- net at U1.68 (VCAP): now also C28.2
- net at U1.103 (VCAP), U1.140 (VCAP): now also C27.2

Commit message: final?
Other:
- company: SAVILO-AKATE PRODUCTIONS -> (none)
Changed lines of the file:
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@@
 		(date "2026-03-12")
 		(rev "v1")
-		(company "SAVILO-AKATE PRODUCTIONS")
 	)
 	(text "NRESET/BOOT"
