File: board/stm32h755xih3/stm32h755xih3.kicad_pcb (KiCad board)
At the start: 4 copper layers, 40.1 x 55.5 mm, 75 parts, among them IC1 USBLC6-2SC6, IC2 USBLC6-2SC6, IC3 USBLC6-2SC6, IC4 USBLC6-2SC6, IC5 USBLC6-2SC6, IC6 USBLC6-2SC6, IC7 USBLC6-2SC6, IC8 TPS629203QDRLRQ1, IC9 AP2112K-3.3TRG1, J1 HTSW-101-07-G-T, J10 HTSW-101-07-G-T, J11 HTSW-101-07-G-T, J12 HTSW-101-07-G-T, J13 HTSW-101-07-G-T, J14 HTSW-101-07-G-T, J15 HTSW-101-07-G-T, J16 HTSW-101-07-G-T, J17 HTSW-101-07-G-T, J18 Conn_ARM_SWD_TagConnect_TC203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, J2 HTSW-101-07-G-T, J3 HTSW-101-07-G-T, J4 BM06B-GHS-GB-TBT_LF__SN_, J5 BM06B-GHS-GB-TBT_LF__SN_, J6 BM06B-GHS-GB-TBT_LF__SN_, J7 HTSW-101-07-G-T, J8 HTSW-101-07-G-T, J9 10155435-00011LF, U1 STM32H755ZITx, Y1 LFXTAL085880

Commit message: pcb update
Parts:
- removed the C1 at (103.8, 57.5)
- removed the C29 at (132.7, 78.8)
- removed D1, D2: MBR0530T1G, MBR0530T1G:SOD3716X135N
- removed the IC1 at (108.0, 91.9)
- removed IC2, IC3, IC4, IC5, IC6, IC7: USBLC6-2SC6, USBLC6-2SC6:SOT95P280X145-6N
- removed IC8: TPS629203QDRLRQ1, TPS629203QDRLRQ1:SOTFL50P160X60-8N
- removed the J1 at (101.2, 53.0)
- removed the J5 at (132.5, 97.8)
- removed the J6 at (119.6, 97.8)
- removed the L1 at (107.3, 61.4)
- removed the R1 at (132.2, 91.1)
- removed the R2 at (101.9, 60.0)
- removed the R3 at (132.2, 85.1)
- added C28: CC0603JRX7R9BB104, 06035C3R9CAT2A:CAPC1608X90N, F.Cu at (204.9, 77.0)
- added C6: CC0603JRX7R9BB104, 06035C3R9CAT2A:CAPC1608X90N, F.Cu at (178.2, 85.3)
- added G***: LOGO, LOGO, B.Cu at (190.3, 76.4)
- added J14: BM06B-GHS-GB-TBT_LF__SN_, BM06B-GHS-GB-TBT_LF__SN_:BM06BGHSGBTBTLFSN, F.Cu at (223.4, 131.4)
- added J17: HTSW-101-07-G-T, HTSW-101-07-G-T:HDRV3W64P254_3X1_254X756X838P, F.Cu at (206.8, 23.4)
- added J4: HTSW-101-07-G-T, HTSW-101-07-G-T:HDRV3W64P254_3X1_254X756X838P, F.Cu at (173.2, 23.4)
- added REF**: TestPoint_Pad_D1.0mm, TestPoint:TestPoint_Pad_D1.0mm, F.Cu at (179.2, 27.5)
- added REF**: TestPoint_Pad_D1.0mm, TestPoint:TestPoint_Pad_D1.0mm, F.Cu at (170.8, 32.1)
- added REF**: TestPoint_Pad_D1.0mm, TestPoint:TestPoint_Pad_D1.0mm, F.Cu at (173.2, 27.5)
- added REF**: TestPoint_Pad_D1.0mm, TestPoint:TestPoint_Pad_D1.0mm, F.Cu at (188.5, 27.5)
- added REF**: TestPoint_Pad_D1.0mm, TestPoint:TestPoint_Pad_D1.0mm, F.Cu at (209.8, 27.5)
- added REF**: TestPoint_Pad_D1.0mm, TestPoint:TestPoint_Pad_D1.0mm, F.Cu at (185.5, 27.5)
- added REF**: TestPoint_Pad_D1.0mm, TestPoint:TestPoint_Pad_D1.0mm, F.Cu at (197.8, 27.5)
- added REF**: TestPoint_Pad_D1.0mm, TestPoint:TestPoint_Pad_D1.0mm, F.Cu at (206.8, 27.5)
- added REF**: TestPoint_Pad_D1.0mm, TestPoint:TestPoint_Pad_D1.0mm, F.Cu at (200.8, 27.5)
- added REF**: TestPoint_Pad_D1.0mm, TestPoint:TestPoint_Pad_D1.0mm, F.Cu at (176.2, 27.5)
- added REF**: TestPoint_Pad_D1.0mm, TestPoint:TestPoint_Pad_D1.0mm, F.Cu at (194.5, 27.5)
- added REF**: TestPoint_Pad_D1.0mm, TestPoint:TestPoint_Pad_D1.0mm, F.Cu at (203.8, 27.5)
- added REF**: TestPoint_Pad_D1.0mm, TestPoint:TestPoint_Pad_D1.0mm, F.Cu at (182.4, 27.5)
- added REF**: TestPoint_Pad_D1.0mm, TestPoint:TestPoint_Pad_D1.0mm, F.Cu at (191.5, 27.5)
- C4: value CL31A226KOCLNNC -> KGM31HR71C105JU; footprint CL31A226KOCLNNC:CAPC3216X95N -> KGM31HR71C105JU:CAPC3216X190N
- J9: value 10155435-00011LF -> BM06B-GHS-GB-TBT_LF__SN_; footprint 10155435-00011LF:AMPHENOL_10155435-00011LF -> BM06B-GHS-GB-TBT_LF__SN_:BM06BGHSGBTBTLFSN
- moved LED1 113.2 mm to (228.2, 20.3)
- moved R1 113.2 mm to (228.1, 18.6)
- moved J16 80.7 mm to (212.9, 23.4)
- moved J13 80.7 mm to (209.8, 23.4)
- moved J12 77.9 mm to (200.7, 23.4)
- moved J15 77.9 mm to (203.7, 23.4)
- moved J3 77.9 mm to (182.4, 23.4)
- moved J7 77.9 mm to (188.5, 23.4)
- moved J8 77.9 mm to (194.6, 23.4)
- moved J10 77.9 mm to (191.5, 23.4)
- moved J11 77.9 mm to (197.6, 23.4)
- moved J2 77.9 mm to (176.2, 23.4)
- moved J5 77.9 mm to (179.3, 23.4)
- moved J6 77.9 mm to (185.4, 23.4)
- moved C4 76.1 mm to (177.4, 87.0), turned to 180 degrees
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- renumbered C2 to C1, C11 to C10, C12 to C11, C13 to C12, C9 to C13, C16 to C15, C18 to C16, C15 to C17, C19 to C18, C17 to C19, C3 to C2, C27 to C26, C26 to C27, C28 to C29, C5 to C3, C33 to C32, C32 to C33, C6 to C5, C8 to C7, C10 to C8, C7 to C9, IC9 to IC1, J4 to J1, J12 to J10, J13 to J11, J14 to J12, J15 to J13, J16 to J15, J17 to J16, J7 to J5, J8 to J6, J10 to J7, J11 to J8, L2 to L1, R4 to R1, R5 to R2, R6 to R3, R7 to R4
Connections:
- C1 pad 1: 5VUSB -> Net-(IC1-EN)
- C17 pad 1: VCAP -> Net-(C17-Pad1)
- C19 pad 1: VCAP -> Net-(C19-Pad1)
- C2 pad 1: 5VUSB -> Net-(IC1-EN)
- C26 pad 1: 3V3USB -> 3V3
- C3 pad 1: Net-(D2-A) -> 3V3
- C4 pad 1: Net-(D1-A) -> 3V3
- IC1 pad 1: 5VUSB -> Net-(IC1-EN)
- IC1 pad 3: 5VUSB -> Net-(IC1-EN)
- IC1 pad 5: Net-(D2-A) -> 3V3
- J1 pad 2: Net-(IC2-I/O2_1) -> TXD1
- J1 pad 3: Net-(IC2-I/O1_1) -> RXD1
- J1 pad 4: Net-(IC1-I/O2_1) -> unconnected-(J1-Pad4)
- J1 pad 5: Net-(IC1-I/O1_1) -> unconnected-(J1-Pad5)
- J12 pad 1: STM32B -> STM32Α1/2
- J13 pad 1: D+ -> STM32D1/2
- J15 pad 1: STM32C -> STM32B1/2
- J16 pad 1: STM32E -> STM32E1/2
- U1 pad 100: D+ -> STM32D1/2
- U1 pad 101: D- -> STM32D1/2
- U1 pad 103: VCAP -> Net-(C19-Pad1)
- U1 pad 109: unconnected-(U1-PC10-Pad109) -> TXD3
- U1 pad 110: unconnected-(U1-PC11-Pad110) -> RXD3
- U1 pad 115: CTS1 -> unconnected-(U1-PD3-Pad115)
- U1 pad 116: RTS1 -> unconnected-(U1-PD4-Pad116)
- U1 pad 117: TXD1 -> TXD2
- U1 pad 120: RXD1 -> RXD2
- U1 pad 122: RXD2 -> unconnected-(U1-PG9-Pad122)
- U1 pad 125: RTS2 -> unconnected-(U1-PG12-Pad125)
- U1 pad 126: CTS2 -> unconnected-(U1-PG13-Pad126)
- U1 pad 127: TXD2 -> unconnected-(U1-PG14-Pad127)
- U1 pad 133: unconnected-(U1-PB6-Pad133) -> TXD1
- U1 pad 134: unconnected-(U1-PB7-Pad134) -> RXD1
- U1 pad 140: VCAP -> Net-(C19-Pad1)
- U1 pad 20: RXD3 -> unconnected-(U1-PF6-Pad20)
- U1 pad 21: TXD3 -> unconnected-(U1-PF7-Pad21)
- U1 pad 22: RTS3 -> unconnected-(U1-PF8-Pad22)
- U1 pad 23: CTS3 -> unconnected-(U1-PF9-Pad23)
- U1 pad 68: VCAP -> Net-(C17-Pad1)
- U1 pad 86: STM32E -> STM32E1/2
- U1 pad 87: unconnected-(U1-PG7-Pad87) -> STM32E1/2
- U1 pad 90: 5VUSB -> unconnected-(U1-VDD50_USB-Pad90)
- U1 pad 91: 3V3USB -> 3V3
- U1 pad 94: unconnected-(U1-PC7-Pad94) -> STM32Α1/2
- U1 pad 95: STM32B -> STM32B1/2
- U1 pad 97: unconnected-(U1-PA8-Pad97) -> STM32B1/2
- U1 pad 98: STM32C -> STM32C1/2
- U1 pad 99: unconnected-(U1-PA10-Pad99) -> STM32C1/2
Routing:
- net 3V3: track 61.6 -> 164.7 mm, vias 112 -> 118
- net TESTLED: track 0.00 -> 93.5 mm, vias 0 -> 2
- net STM32E1/2: track 0.00 -> 71.9 mm, vias 0 -> 2
- net APU2A: track 37.3 -> 108.8 mm, vias 4 -> 2
- net STM32Α1/2: track 0.00 -> 71.2 mm, vias 0 -> 2
- net STM32B1/2: track 0.00 -> 69.1 mm, vias 0 -> 2
- net STM32C1/2: track 0.00 -> 67.8 mm, vias 0 -> 2
- net STM32D1/2: track 0.00 -> 66.6 mm, vias 0 -> 2
- net APU1A: track 46.9 -> 98.1 mm, vias 4 -> 0
- net 5VUSB: track 47.0 -> 0.00 mm, vias 5 -> 0
- net APU2B: track 31.4 -> 74.5 mm
- net RXD1: track 31.9 -> 74.8 mm, vias 4 -> 2
- net TXD3: track 32.5 -> 74.6 mm, vias 8 -> 2
- net RXD3: track 34.0 -> 74.7 mm, vias 6 -> 2
- net APU2C: track 37.7 -> 77.6 mm
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Other:
- board size 40.1 x 55.5 mm -> 80 x 120 mm
- board text added: "C25"
- board text added: "C3"
- board text added: "E"
- board text added: "FABRICATION NOTES: 1. MATERIAL: FR4 150TG 2. TOTAL THICKNESS: 1.55mm +/- 10% 3. SURFACE FINISH: ENIG (Ni/Au) 4. STANDARD: IPC-A-600 CLASS 2"
- board text added: "SWD"
- board text added: "UART1"
- board text added: "UART2"
- board text added: "UART3"

Commit message: board updates
Parts:
- removed the C13 at (173.8, 74.8)
- removed the C22 at (178.6, 75.3)
- removed the C9 at (175.0, 69.6)
- removed the J1 at (159.5, 131.5)
- removed the J14 at (223.4, 131.4)
- removed the J9 at (191.5, 131.3)
- removed L1: SRP3212-2R2M, SRP3212-2R2M:INDC2520X100N
- removed the REF** at (179.2, 27.5)
- removed the REF** at (170.8, 32.1)
- removed the REF** at (173.2, 27.5)
- removed the REF** at (188.5, 27.5)
- removed the REF** at (209.8, 27.5)
- removed the REF** at (185.5, 27.5)
- removed the REF** at (197.8, 27.5)
- removed the REF** at (206.8, 27.5)
- removed the REF** at (200.8, 27.5)
- removed the REF** at (176.2, 27.5)
- removed the REF** at (194.5, 27.5)
- removed the REF** at (203.8, 27.5)
- removed the REF** at (182.4, 27.5)
- removed the REF** at (191.5, 27.5)
- added J11: 205957-0671, 205957-0671:2059570671, F.Cu at (191.5, 131.4)
- added J17: 205957-0671, 205957-0671:2059570671, F.Cu at (223.4, 131.4)
- added J6: 205957-0671, 205957-0671:2059570671, F.Cu at (159.4, 131.4)
- added REF**: TestPoint_Pad_D1.0mm, TestPoint:TestPoint_Pad_D1.0mm, F.Cu at (191.5, 27.4)
- added REF**: TestPoint_Pad_D1.0mm, TestPoint:TestPoint_Pad_D1.0mm, F.Cu at (194.6, 27.4)
- added REF**: TestPoint_Pad_D1.0mm, TestPoint:TestPoint_Pad_D1.0mm, F.Cu at (173.2, 27.4)
- added REF**: TestPoint_Pad_D1.0mm, TestPoint:TestPoint_Pad_D1.0mm, F.Cu at (176.3, 27.4)
- added REF**: TestPoint_Pad_D1.0mm, TestPoint:TestPoint_Pad_D1.0mm, F.Cu at (179.3, 27.4)
- added REF**: TestPoint_Pad_D1.0mm, TestPoint:TestPoint_Pad_D1.0mm, F.Cu at (200.7, 27.4)
- added REF**: TestPoint_Pad_D1.0mm, TestPoint:TestPoint_Pad_D1.0mm, F.Cu at (185.4, 27.4)
- added REF**: TestPoint_Pad_D1.0mm, TestPoint:TestPoint_Pad_D1.0mm, F.Cu at (212.9, 27.4)
- added REF**: TestPoint_Pad_D1.0mm, TestPoint:TestPoint_Pad_D1.0mm, F.Cu at (197.6, 27.4)
- added REF**: TestPoint_Pad_D1.0mm, TestPoint:TestPoint_Pad_D1.0mm, F.Cu at (170.8, 32.1)
- added REF**: TestPoint_Pad_D1.0mm, TestPoint:TestPoint_Pad_D1.0mm, F.Cu at (203.7, 27.4)
- added REF**: TestPoint_Pad_D1.0mm, TestPoint:TestPoint_Pad_D1.0mm, F.Cu at (206.8, 27.4)
- added REF**: TestPoint_Pad_D1.0mm, TestPoint:TestPoint_Pad_D1.0mm, F.Cu at (188.5, 27.4)
- added REF**: TestPoint_Pad_D1.0mm, TestPoint:TestPoint_Pad_D1.0mm, F.Cu at (182.4, 27.4)
- added REF**: TestPoint_Pad_D1.0mm, TestPoint:TestPoint_Pad_D1.0mm, F.Cu at (209.8, 27.4)
- C26: renamed from C31; value 06035C3R9CAT2A -> GRM1555C1H8R0DA01D; footprint 06035C3R9CAT2A:CAPC1608X90N -> GRM1555C1H8R0DA01D:CAPC1005X70N
- C28: renamed from C33; value 06035C3R9CAT2A -> GRM1555C1H8R0DA01D; footprint 06035C3R9CAT2A:CAPC1608X90N -> GRM1555C1H8R0DA01D:CAPC1005X70N
- J18: value Conn_ARM_SWD_TagConnect_TC2030-NL -> 205957-0671; footprint Connector:Tag-Connect_TC2030-IDC-NL_2x03_P1.27mm_Vertical -> 205957-0671:2059570671
- turned C28 to 180 degrees
- renumbered C11 to C10, C12 to C11, C25 to C12, C14 to C13, C15 to C14, C16 to C15, C18 to C16, C27 to C17, C20 to C18, C29 to C19, C21 to C20, C30 to C21, C23 to C22, C24 to C23, C26 to C24, C28 to C25, C32 to C27, C19 to C29, C17 to C30, C5 to C4, C7 to C5, C4 to C6, C8 to C7, C6 to C8, C10 to C9, J2 to J1, J11 to J10, J15 to J14, J16 to J15, J17 to J16, J3 to J2, J4 to J3, J5 to J4, J6 to J5, J10 to J9
Connections:
- net APU1A renamed AP1_1
- net APU1B renamed AP1_2
- net APU1C renamed AP1_3
- net APU1D renamed AP1_4
- net APU2A renamed AP2_1
- net APU2B renamed AP2_2
- net APU2C renamed AP2_3
- net APU2D renamed AP2_4
- C28 pad 1: OSC1 -> GND
- C28 pad 2: GND -> OSC1
- J18 pad 2: SWDIO -> NRESET
- J18 pad 3: NRESET -> SWCLK
- J18 pad 4: SWCLK -> SWDIO
- J18 pad 5: GND -> SWO
- J18 pad 6: SWO -> GND
- U1 pad 15: VLXSMPS -> unconnected-(U1-VLXSMPS-Pad15)
- U1 pad 16: 3V3 -> GND
- U1 pad 17: VFBSMPS -> GND
Routing:
- net VFBSMPS: track 15.9 -> 0.00 mm, vias 2 -> 0
- net VLXSMPS: track 15.5 -> 0.00 mm, vias 2 -> 0
- net 3V3: track 164.7 -> 149.5 mm, vias 118 -> 70
- net TXD3: track 74.6 -> 84.8 mm
- net TXD2: track 64.6 -> 73.9 mm
- net TXD1: track 74.9 -> 82.5 mm
- net SWDIO: track 62.8 -> 55.8 mm, vias 2 -> 4
- net SWCLK: track 62.9 -> 58.0 mm
- net SWO: track 50.6 -> 48.2 mm
- net NRESET: track 36.0 -> 34.9 mm, vias 2 -> 4
- net AP2_4: track 58.1 -> 57.4 mm
- net RXD3: track 74.7 -> 74.0 mm
- net GND: vias 1776 -> 133
Other:
- board text added: "1"
- board text added: "2"
- board text added: "3"
- board text added: "4"
- board text added: "5"
- board text added: "AP1_1"
- board text added: "AP1_2"
- board text added: "AP1_3"
- board text added: "AP1_4"
- board text added: "AP2_1"
- board text added: "AP2_2"
- board text added: "AP2_3"
- board text added: "AP2_4"
- board text removed: "1A"
- board text removed: "1B"
- board text removed: "1C"
- board text removed: "1D"
- board text removed: "2A"
- board text removed: "2B"
- board text removed: "2C"
- board text removed: "2D"
- board text removed: "A"
- board text removed: "B"
- board text removed: "C"
- board text removed: "D"
- board text removed: "E"

Commit message: board clearance
Routing:
- net TESTLED: track 93.5 -> 92.5 mm
- net STM32C1/2: track 67.8 -> 68.5 mm
- net STM32D1/2: track 66.6 -> 67.3 mm
- net SWCLK: track 58.0 -> 58.6 mm

Commit message: board final???
Parts:
- removed C29, C30: 12065C225JAT2A, 12065C225JAT2A:CAPC3216X229N
- removed G***: LOGO, LOGO
- removed the REF** at (191.5, 27.4)
- removed the REF** at (194.6, 27.4)
- removed the REF** at (173.2, 27.4)
- removed the REF** at (176.3, 27.4)
- removed the REF** at (179.3, 27.4)
- removed the REF** at (200.7, 27.4)
- removed the REF** at (185.4, 27.4)
- removed the REF** at (212.9, 27.4)
- removed the REF** at (197.6, 27.4)
- removed the REF** at (170.8, 32.1)
- removed the REF** at (203.7, 27.4)
- removed the REF** at (206.8, 27.4)
- removed the REF** at (188.5, 27.4)
- removed the REF** at (182.4, 27.4)
- removed the REF** at (209.8, 27.4)
- added REF**: TestPoint_Pad_D1.0mm, TestPoint:TestPoint_Pad_D1.0mm, F.Cu at (103.7, 51.9)
- added REF**: TestPoint_Pad_D1.0mm, TestPoint:TestPoint_Pad_D1.0mm, F.Cu at (113.0, 51.9)
- added REF**: TestPoint_Pad_D1.0mm, TestPoint:TestPoint_Pad_D1.0mm, F.Cu at (128.5, 51.9)
- added REF**: TestPoint_Pad_D1.0mm, TestPoint:TestPoint_Pad_D1.0mm, F.Cu at (125.4, 51.9)
- added REF**: TestPoint_Pad_D1.0mm, TestPoint:TestPoint_Pad_D1.0mm, F.Cu at (122.3, 51.9)
- added REF**: TestPoint_Pad_D1.0mm, TestPoint:TestPoint_Pad_D1.0mm, F.Cu at (100.6, 51.9)
- added REF**: TestPoint_Pad_D1.0mm, TestPoint:TestPoint_Pad_D1.0mm, F.Cu at (109.9, 51.9)
- added REF**: TestPoint_Pad_D1.0mm, TestPoint:TestPoint_Pad_D1.0mm, F.Cu at (106.8, 51.9)
- added REF**: TestPoint_Pad_D1.0mm, TestPoint:TestPoint_Pad_D1.0mm, F.Cu at (132.1, 51.9)
- added REF**: TestPoint_Pad_D1.0mm, TestPoint:TestPoint_Pad_D1.0mm, F.Cu at (116.1, 51.9)
- added REF**: TestPoint_Pad_D1.0mm, TestPoint:TestPoint_Pad_D1.0mm, F.Cu at (94.4, 51.9)
- added REF**: TestPoint_Pad_D1.0mm, TestPoint:TestPoint_Pad_D1.0mm, F.Cu at (97.5, 51.9)
- added REF**: TestPoint_Pad_D1.0mm, TestPoint:TestPoint_Pad_D1.0mm, F.Cu at (119.2, 51.9)
- C17, C6: value KGM31HR71C105JU -> CC0603JRX7R9BB104; footprint KGM31HR71C105JU:CAPC3216X190N -> 06035C3R9CAT2A:CAPC1608X90N
- C19, C2, C21, C3: value KGM31HR71C105JU -> C0603X105J4RACTU; footprint KGM31HR71C105JU:CAPC3216X190N -> C0603X105J4RACTU:C0603
- C23, C8: value CC0603JRX7R9BB104 -> C0603X105J4RACTU; footprint 06035C3R9CAT2A:CAPC1608X90N -> C0603X105J4RACTU:C0603
- C24: value KGM31HR71C105JU -> GRM1555C1H8R0DA01D; footprint KGM31HR71C105JU:CAPC3216X190N -> GRM1555C1H8R0DA01D:CAPC1005X70N
- C27: value CC0603JRX7R9BB104 -> 12065C225JAT2A; footprint 06035C3R9CAT2A:CAPC1608X90N -> 12065C225JAT2A:CAPC3216X229N
- C28: value GRM1555C1H8R0DA01D -> 12065C225JAT2A; footprint GRM1555C1H8R0DA01D:CAPC1005X70N -> 12065C225JAT2A:CAPC3216X229N
- C4: value MLASG168BB5475KTNA01 -> CC0603JRX7R9BB104; footprint MLASG168BB5475KTNA01:CAPC1709X100N -> 06035C3R9CAT2A:CAPC1608X90N
- C5: value CC0603JRX7R9BB104 -> MLASG168BB5475KTNA01; footprint 06035C3R9CAT2A:CAPC1608X90N -> MLASG168BB5475KTNA01:CAPC1709X100N
- J11, J17, J6: value 205957-0671 -> HTSW-101-07-G-T; footprint 205957-0671:2059570671 -> HTSW-101-07-G-T:HDRV3W64P254_3X1_254X756X838P
- J14, J4, J9: value HTSW-101-07-G-T -> 53047-0610; footprint HTSW-101-07-G-T:HDRV3W64P254_3X1_254X756X838P -> 53047-0610:530470610
- J18: value 205957-0671 -> 53047-0610; footprint 205957-0671:2059570671 -> 53047-0610:530470610
- Y1: value LFXTAL085880 -> 830059082
- moved J14 168.3 mm to (90.9, 148.2)
- moved J17 150.7 mm to (102.2, 42.0)
- moved J9 144.6 mm to (118.6, 148.2)
- moved J4 129.5 mm to (145.0, 148.2)
- moved C25 124.8 mm to (86.0, 114.8)
- moved LED1 123.5 mm to (115.8, 71.5), turned to 90 degrees
- moved R1 122.6 mm to (117.6, 71.5), turned to 90 degrees
- moved J13 112.3 mm to (99.1, 42.0), turned to 180 degrees
- moved J15 109.2 mm to (105.3, 42.0), turned to 180 degrees
- moved J11 108.5 mm to (130.1, 42.0)
- moved C16 106.9 mm to (100.7, 98.7), turned to 90 degrees
- moved C15 104.7 mm to (101.3, 93.3), turned to 180 degrees
- moved C18 104.3 mm to (111.1, 112.9), turned to -90 degrees
- moved C17 102.0 mm to (101.0, 108.1), turned to 180 degrees
- moved C19 101.9 mm to (107.0, 84.5), turned to 90 degrees
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Connections:
- C2 pad 1: Net-(IC1-EN) -> GND
- C2 pad 2: GND -> Net-(IC1-EN)
- C24 pad 1: 3V3 -> OSC2
- C25 pad 1: 3V3 -> NRESET
- C26 pad 1: OSC2 -> GND
- C26 pad 2: GND -> OSC1
- C27 pad 1: NRESET -> Net-(C27-Pad1)
- C28 pad 1: GND -> Net-(C28-Pad1)
- C28 pad 2: OSC1 -> GND
- C3 pad 1: 3V3 -> GND
- C3 pad 2: GND -> 3V3
- J10 pad 1: AP2_4 -> AP2_2
- J11 pad 1: GND -> AP2_4
- J11 pad 3: unconnected-(J11-Pad3) -> GND
- J14 pad 1: STM32B1/2 -> GND
- J14 pad 3: GND -> unconnected-(J14-Pad3)
- J15 pad 1: STM32E1/2 -> STM32B1/2
- J16 pad 1: STM32C1/2 -> STM32E1/2
- J17 pad 1: GND -> STM32C1/2
- J17 pad 3: unconnected-(J17-Pad3) -> GND
- J4 pad 1: AP1_2 -> GND
- J4 pad 3: GND -> unconnected-(J4-Pad3)
- J5 pad 1: AP1_4 -> AP1_2
- J6 pad 1: GND -> AP1_4
- J6 pad 3: unconnected-(J6-Pad3) -> GND
- J9 pad 1: AP2_2 -> GND
- J9 pad 3: GND -> unconnected-(J9-Pad3)
- U1 pad 103: Net-(C29-Pad1) -> Net-(C27-Pad1)
- U1 pad 140: Net-(C29-Pad1) -> Net-(C27-Pad1)
- U1 pad 68: Net-(C30-Pad1) -> Net-(C28-Pad1)
- U1 pad 90: unconnected-(U1-VDD50_USB-Pad90) -> 3V3
Routing:
- net TESTLED: track 92.5 -> 16.0 mm, vias 2 -> 0
- net AP2_1: track 108.8 -> 48.1 mm, vias 2 -> 0
- net AP1_3: track 45.5 -> 97.1 mm, vias 2 -> 0
- net TXD3: track 84.8 -> 46.9 mm, vias 2 -> 0
- net TXD2: track 73.9 -> 40.4 mm, vias 2 -> 0
- net TXD1: track 82.5 -> 52.8 mm
- net SWCLK: track 58.6 -> 29.7 mm, vias 4 -> 0
- net SWDIO: track 55.8 -> 28.6 mm, vias 4 -> 1
- net 3V3: track 149.7 -> 123.0 mm, vias 70 -> 38
- net RXD3: track 74.0 -> 47.3 mm, vias 2 -> 0
- net Net-(C29-Pad1): track 24.9 -> 0.00 mm
- net RXD2: track 65.0 -> 40.8 mm, vias 2 -> 0
- net Net-(C27-Pad1): track 0.00 -> 22.0 mm
- net RXD1: track 74.9 -> 53.0 mm
- net AP1_1: track 98.1 -> 77.2 mm
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Other:
- board text added: "APU-MUX v1"
- board text added: "eXeLIIgence"
- board text removed: "1"
- board text removed: "2"
- board text removed: "3"
- board text removed: "4"
- board text removed: "5"
- board text removed: "AP1_1"
- board text removed: "AP1_2"
- board text removed: "AP1_3"
- board text removed: "AP1_4"
- board text removed: "AP2_1"
- board text removed: "AP2_2"
- board text removed: "AP2_3"
- board text removed: "AP2_4"
- board text removed: "APU-MUX v1 CHRKARAS"
- board text removed: "C25"
- board text removed: "C3"
- board text removed: "PWR"
- board text removed: "PWR LED"
- board text removed: "SWD"
- board text removed: "TEST LED"

Commit message: final??
Parts:
- removed REF** (x13): TestPoint_Pad_D1.0mm, TestPoint:TestPoint_Pad_D1.0mm
- C27, C28: value 12065C225JAT2A -> 0603YC225MAT2A; footprint 12065C225JAT2A:CAPC3216X229N -> 0603YC225MAT2A:CAPC1608X90N
- moved C27 0.73 mm to (121.6, 112.7), turned to 90 degrees
- moved C28 0.57 mm to (109.6, 85.0), turned to -90 degrees
Connections:
- C27 pad 1: Net-(C27-Pad1) -> GND
- C27 pad 2: GND -> Net-(C27-Pad2)
- C28 pad 1: Net-(C28-Pad1) -> GND
- C28 pad 2: GND -> Net-(C28-Pad2)
- U1 pad 103: Net-(C27-Pad1) -> Net-(C27-Pad2)
- U1 pad 140: Net-(C27-Pad1) -> Net-(C27-Pad2)
- U1 pad 68: Net-(C28-Pad1) -> Net-(C28-Pad2)
Routing:
- net Net-(C27-Pad2): track 0.00 -> 22.0 mm
- net Net-(C27-Pad1): track 22.0 -> 0.00 mm
- net Net-(C28-Pad2): track 0.00 -> 3.56 mm
- net Net-(C28-Pad1): track 3.56 -> 0.00 mm
- net AP1_1: track 77.2 -> 78.0 mm

Commit message: final?
Other:
- board text added: "AP1_1"
- board text added: "AP1_2"
- board text added: "AP1_3"
- board text added: "AP1_4"
- board text added: "AP2_1"
- board text added: "AP2_2"
- board text added: "AP2_3"
- board text added: "AP2_4"
- board text added: "BOOT"
- board text added: "NRST"
- board text added: "OUT_1"
- board text added: "OUT_2"
- board text added: "OUT_3"
- board text added: "OUT_4"
- board text added: "OUT_5"
- board text added: "PWR"
- board text added: "PWR LED"
- board text added: "SWD"
- board text added: "TEST LED"
Changed lines of the file:
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@@
 		(layer "Edge.Cuts")
+	)
+	(gr_text "AP2_3"
+		(at 120.75 52.25 90)
+		(layer "F.SilkS")
+		(effects
+			(font
+				(size 1.5 1.5)
+				(thickness 0.3)
+				(bold yes)
+			)
+		)
+	)
+	(gr_text "TEST\nLED"
+		(at 111.7 71.55 0)
+		(layer "F.SilkS")
+		(effects
+			(font
+				(size 1.5 1.5)
+				(thickness 0.3)
+				(bold yes)
+			)
+		)
+	)
+	(gr_text "AP2_2"
+		(at 111.5 52.25 90)
+		(layer "F.SilkS")
+		(effects
+			(font
+				(size 1.5 1.5)
+				(thickness 0.3)
+				(bold yes)
+			)
+		)
+	)
+	(gr_text "AP2_4"
+		(at 130.25 52.25 90)
+		(layer "F.SilkS")
+		(effects
+			(font
+				(size 1.5 1.5)
+				(thickness 0.3)
+				(bold yes)
+			)
+		)
+	)
+	(gr_text "OUT_2"
+		(at 105.25 52.25 90)
+		(layer "F.SilkS")
+		(effects
+			(font
+				(size 1.5 1.5)
+				(thickness 0.3)
+				(bold yes)
+			)
+		)
+	)
+	(gr_text "AP1_3"
+		(at 133.5 52.25 90)
+		(layer "F.SilkS")
+		(effects
+			(font
+				(size 1.5 1.5)
+				(thickness 0.3)
+				(bold yes)
+			)
+		)
+	)
+	(gr_text "AP2_1"
+		(at 127 52.25 90)
+		(layer "F.SilkS")
+		(effects
+			(font
+				(size 1.5 1.5)
+				(thickness 0.3)
+				(bold yes)
+			)
+		)
+	)
+	(gr_text "AP1_1"
+		(at 123.85 52.25 90)
+		(layer "F.SilkS")
+		(effects
+			(font
+				(size 1.5 1.5)
+				(thickness 0.3)
+				(bold yes)
+			)
+		)
 	)
 	(gr_text "UART3"
@@
 		)
 	)
+	(gr_text "AP1_4"
+		(at 117.5 52.25 90)
+		(layer "F.SilkS")
+		(effects
+			(font
+				(size 1.5 1.5)
+				(thickness 0.3)
+				(bold yes)
+			)
+		)
+	)
+	(gr_text "SWD"
+		(at 76 109 0)
+		(layer "F.SilkS")
+		(effects
+			(font
+				(size 3 3)
+				(thickness 0.75)
+				(bold yes)
+			)
+			(justify left bottom)
+		)
+	)
 	(gr_text "UART2"
 		(at 108.1 145.75 0)
@@
 			)
 			(justify left bottom)
+		)
+	)
+	(gr_text "PWR\nLED"
+		(at 84.2 61.9 0)
+		(layer "F.SilkS")
+		(effects
+			(font
+				(size 1.5 1.5)
+				(thickness 0.3)
+				(bold yes)
+			)
+		)
+	)
+	(gr_text "OUT_3"
+		(at 102.25 52.25 90)
+		(layer "F.SilkS")
+		(effects
+			(font
+				(size 1.5 1.5)
+				(thickness 0.3)
+				(bold yes)
+			)
 		)
 	)
@@
 			)
 		)
+	)
+	(gr_text "OUT_5"
+		(at 114.5 52.25 90)
+		(layer "F.SilkS")
+		(effects
+			(font
+				(size 1.5 1.5)
+				(thickness 0.3)
+				(bold yes)
+			)
+		)
+	)
+	(gr_text "NRST"
+		(at 85 120.25 90)
+		(layer "F.SilkS")
+		(effects
+			(font
+				(size 1 1)
+				(thickness 0.25)
+				(bold yes)
+			)
+			(justify left bottom)
+		)
+	)
+	(gr_text "AP1_2"
+		(at 96 52.25 90)
+		(layer "F.SilkS")
+		(effects
+			(font
+				(size 1.5 1.5)
+				(thickness 0.3)
+				(bold yes)
+			)
+		)
+	)
+	(gr_text "PWR"
+		(at 93 52 90)
+		(layer "F.SilkS")
+		(effects
+			(font
+				(size 1.5 1.5)
+				(thickness 0.3)
+				(bold yes)
+			)
+		)
+	)
+	(gr_text "BOOT"
+		(at 118.25 115.5 90)
+		(layer "F.SilkS")
+		(effects
+			(font
+				(size 1 1)
+				(thickness 0.25)
+				(bold yes)
+			)
+			(justify left bottom)
+		)
+	)
+	(gr_text "OUT_1"
+		(at 108.25 52 90)
+		(layer "F.SilkS")
+		(effects
+			(font
+				(size 1.5 1.5)
+				(thickness 0.3)
+				(bold yes)
+			)
+		)
+	)
+	(gr_text "OUT_4"
+		(at 99 52.25 90)
+		(layer "F.SilkS")
+		(effects
+			(font
+				(size 1.5 1.5)
+				(thickness 0.3)
+				(bold yes)
+			)
+		)
