File: board/stm32h755xih3/stm32h755xih3.kicad_pcb (KiCad board)
At the start: 4 copper layers, 80 x 120 mm, 55 parts, among them IC1 AP2112K-3.3TRG1, J1 HTSW-101-07-G-T, J10 HTSW-101-07-G-T, J11 HTSW-101-07-G-T, J12 HTSW-101-07-G-T, J13 HTSW-101-07-G-T, J14 53047-0610, J15 HTSW-101-07-G-T, J16 HTSW-101-07-G-T, J17 HTSW-101-07-G-T, J18 53047-0610, J2 HTSW-101-07-G-T, J3 HTSW-101-07-G-T, J4 53047-0610, J5 HTSW-101-07-G-T, J6 HTSW-101-07-G-T, J7 HTSW-101-07-G-T, J8 HTSW-101-07-G-T, J9 53047-0610, U1 STM32H755ZITx, Y1 830059082

Commit message: final?
Parts:
- added REF**: TestPoint_Pad_D1.0mm, TestPoint:TestPoint_Pad_D1.0mm, F.Cu at (104.0, 40.6)
- added REF**: TestPoint_Pad_D1.0mm, TestPoint:TestPoint_Pad_D1.0mm, F.Cu at (135.0, 40.8)
- added REF**: TestPoint_Pad_D1.0mm, TestPoint:TestPoint_Pad_D1.0mm, F.Cu at (125.7, 40.7)
- added REF**: TestPoint_Pad_D1.0mm, TestPoint:TestPoint_Pad_D1.0mm, F.Cu at (128.8, 40.7)
- added REF**: TestPoint_Pad_D1.0mm, TestPoint:TestPoint_Pad_D1.0mm, F.Cu at (89.3, 50.8)
- added REF**: TestPoint_Pad_D1.0mm, TestPoint:TestPoint_Pad_D1.0mm, F.Cu at (100.8, 40.6)
- added REF**: TestPoint_Pad_D1.0mm, TestPoint:TestPoint_Pad_D1.0mm, F.Cu at (116.4, 40.7)
- added REF**: TestPoint_Pad_D1.0mm, TestPoint:TestPoint_Pad_D1.0mm, F.Cu at (97.8, 40.6)
- added REF**: TestPoint_Pad_D1.0mm, TestPoint:TestPoint_Pad_D1.0mm, F.Cu at (119.5, 40.7)
- added REF**: TestPoint_Pad_D1.0mm, TestPoint:TestPoint_Pad_D1.0mm, F.Cu at (131.9, 40.7)
- added REF**: TestPoint_Pad_D1.0mm, TestPoint:TestPoint_Pad_D1.0mm, F.Cu at (107.0, 40.6)
- added REF**: TestPoint_Pad_D1.0mm, TestPoint:TestPoint_Pad_D1.0mm, F.Cu at (113.3, 40.7)
- added REF**: TestPoint_Pad_D1.0mm, TestPoint:TestPoint_Pad_D1.0mm, F.Cu at (110.2, 40.7)
- added REF**: TestPoint_Pad_D1.0mm, TestPoint:TestPoint_Pad_D1.0mm, F.Cu at (122.6, 40.7)
- moved J10 2.42 mm to (113.3, 43.6)
- moved J11 2.42 mm to (131.9, 43.6)
- moved J13 2.42 mm to (100.9, 43.6)
- moved J15 2.42 mm to (107.1, 43.6)
- moved J16 2.42 mm to (116.4, 43.6)
- moved J2 2.42 mm to (135.0, 43.6)
- moved J5 2.42 mm to (97.8, 43.6)
- moved J8 2.42 mm to (122.6, 43.6)
- moved J1 2.42 mm to (125.7, 43.6)
- moved J12 2.42 mm to (110.2, 43.6)
- moved J17 2.42 mm to (104.0, 43.6)
- moved J3 2.42 mm to (94.6, 43.6)
- moved J6 2.42 mm to (119.5, 43.6)
- moved J7 2.42 mm to (128.8, 43.6)
Routing:
- net 3V3: track 123.0 -> 126.4 mm
- net STM32D1/2: track 71.5 -> 73.7 mm
- net STM32B1/2: track 72.5 -> 74.6 mm
- net STM32C1/2: track 71.8 -> 73.9 mm
- net AP2_2: track 73.0 -> 75.0 mm
- net AP2_3: track 69.3 -> 71.3 mm
- net AP1_1: track 78.0 -> 80.0 mm
- net AP1_4: track 71.7 -> 73.7 mm
- net STM32Α1/2: track 71.0 -> 73.0 mm
- net STM32E1/2: track 72.7 -> 74.7 mm
- net AP2_1: track 48.1 -> 50.0 mm
- net AP1_2: track 76.1 -> 77.6 mm
- net AP1_3: track 97.1 -> 97.9 mm
- net AP2_4: track 75.5 -> 76.0 mm
- net GND: vias 22 -> 29

Commit message: final???
Parts:
- added REF**: ESD-Logo_6.6x6mm_SilkScreen, Symbol:ESD-Logo_6.6x6mm_SilkScreen, F.Cu at (145.6, 125.4)
